File: PCB/kikad/kikad.kicad_pcb (KiCad board)
At the start: 2 copper layers, 228.6 x 137.2 mm, 207 parts, among them M1 SSOP-24_5.3x8.2mm_P0.65mm, M2 SSOP-24_5.3x8.2mm_P0.65mm

Commit message: motor driver beginning
Parts:
- added C2: 10µF, 0805-NO, F.Cu at (123.7, 31.8)
- added m1: PinHeader_1x02_P1.00mm_Vertical, Connector_PinHeader_1.00mm:PinHeader_1x02_P1.00mm_Vertical, F.Cu at (122.1, 34.2)
- added m2: PinHeader_1x02_P1.00mm_Vertical, Connector_PinHeader_1.00mm:PinHeader_1x02_P1.00mm_Vertical, F.Cu at (125.6, 34.2)
- added m3: PinHeader_1x02_P1.00mm_Vertical, Connector_PinHeader_1.00mm:PinHeader_1x02_P1.00mm_Vertical, F.Cu at (122.1, 38.3)
- added m4: PinHeader_1x02_P1.00mm_Vertical, Connector_PinHeader_1.00mm:PinHeader_1x02_P1.00mm_Vertical, F.Cu at (125.6, 38.3)
- moved M2 16.3 mm to (144.1, 36.3)
- moved Serial 13.0 mm to (153.0, 34.5)
Routing:
- net (no net): track 1578.2 -> 3004.7 mm, vias 0 -> 10
Other:
- outline, holes or cut-outs redrawn

Commit message: more
Parts:
- added C2: 10µF, 0805-NO, F.Cu at (144.3, 30.9)
- moved C2 0.30 mm to (124.0, 31.9)
Routing:
- net (no net): track 3004.7 -> 3402.7 mm, vias 10 -> 15
